File: de10-lite-ram-rom.sch (KiCad schematic (older format))
At the start: 14 parts, among them J1 Conn_02x20_Odd_Even, U1 IS61C5128AS-25TLI, U2 SST39SF040, U3 74LVC2G04

Commit message: fixed labels, tracks, created gerbers
Parts:
- J1: value Conn_02x20_Odd_Even -> DE10-Lite GPIO
Other:
- note added: "512K Flash"
- note added: "512K SRAM"
- moved on the sheet: C1, C2, C3, D1, D2, J1, R1, R2, R3, R4, R5, U1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

Commit message: changed SRAM type
Parts:
- U1: value IS61C5128AS-25TLI -> AS6C4008A-55ZIN; symbol Memory_RAM:IS61C5128AS-25TLI -> Memory_RAM:AS6C4008A-55ZIN
Changed lines of the file:
@@
 ~WR
 $Comp
-L Memory_RAM:IS61C5128AS-25TLI U1
+L Memory_RAM:AS6C4008A-55ZIN U1
 U 1 1 5D78B32A
 P 6100 2650
 F 0 "U1" H 5700 3900 50  0000 C CNN
-F 1 "IS61C5128AS-25TLI" H 6150 2650 50  0000 C CNN
+F 1 "AS6C4008A-55ZIN" H 6150 2650 50  0000 C CNN
 F 2 "Package_SO:TSOP-II-32_21.0x10.2mm_P1.27mm" H 5600 3800 50  0001 C CNN
-F 3 "http://www.issi.com/WW/pdf/61-64C5128AL.pdf" H 6100 2650 50  0001 C CNN
+F 3 "https://www.mouser.com/datasheet/2/12/AS6C4008A-1288404.pdf" H 6100 2650 50  0001 C CNN
 	1    6100 2650
 	1    0    0    -1
@@
 F 1 "74LVC2G04" H 9325 4876 50  0000 C CNN
 F 2 "Package_TO_SOT_SMD:SOT-23-6_Handsoldering" H 9350 4700 50  0001 C CNN
-F 3 "http://www.ti.com/lit/sg/scyt129e/scyt129e.pdf" H 9350 4700 50  0001 C CNN
+F 3 "http://www.ti.com/lit/ds/symlink/sn74lvc2g04.pdf" H 9350 4700 50  0001 C CNN
 	1    9350 4700
 	1    0    0    -1
